File: hw/parts/W5500-EVB-Pico/altium2kicad/W5500-EVB-Pico_V100-PcbDoc.kicad_pcb (KiCad board)
At the start: 2 copper layers, 89 parts, among them J1 J1, J2 J2, J3 J3, P1 P1, P2 P2, Q1 Q1, SW1 SW1, SW2 SW2, U1 U1, U2 U2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

Commit message: w5500-evb-pico footprint
Parts:
- removed C1: C1, CAP-0402
- removed C10: C10, CAP-0402
- removed C11: C11, CAP-0402
- removed C13: C13, CAP-0402
- removed C14: C14, CAP-0402
- removed C2: C2, CAP-0402
- removed C24: C24, CAP-0402
- removed C25: C25, CAP-0402
- removed C26: C26, CAP-0402
- removed C27: C27, CAP-0402
- removed C3: C3, CAP-0402
- removed C32: C32, CAP-0402
- removed C33: C33, CAP-0402
- removed C34: C34, CAP-0402
- removed C37: C37, CAP-0805
- removed C4: C4, CAP-0402
- removed C5: C5, CAP-0402
- removed C6: C6, CAP-0402
- removed C7: C7, CAP-0402
- removed C8: C8, CAP-0402
- removed C9: C9, CAP-0402
- removed D1: D1, SOD-323(1-C,2-A)
- removed L1: L1, IND-0603
- removed LD1: LD1, LED-0603-RED
- removed Q1: Q1, SOT23-3L
- removed R1: R1, RES-0402
- removed R10: R10, RES-0402
- removed R11: R11, RES-0402
- removed R13: R13, RES-0402
- removed R14: R14, RES-0402
- removed R2: R2, RES-0402
- removed R23: R23, RES-0402
- removed R24: R24, RES-0402
- removed R25: R25, RES-0402
- removed R31: R31, RES-0402
- removed R32: R32, RES-0402
- removed R33: R33, RES-0402
- removed R6: R6, RES-0402
- removed R7: R7, RES-0402
- removed R8: R8, RES-0402
- removed R9: R9, RES-0402
- removed SW1: SW1, PTS820
- removed SW2: SW2, PTS820
- removed U1: U1, SOT-23-5L
- removed U2: U2, QFN56(0.4/7X7)
- removed U3: U3, W5500-LQFP48
- removed U4: U4, WSON8(6X5_1.27)
- removed Y1: Y1, OSC-TZ1067B
- removed Y2: Y2, OSC-82J0626
- C12: value C12 -> Ceramic CAP 0402(1005)
- C15: value C15 -> Ceramic CAP 0402(1005)
- C16: value C16 -> Ceramic CAP 0402(1005)
- C17: value C17 -> Ceramic CAP 0402(1005)
- C18: value C18 -> Ceramic CAP 0402(1005)
- C19: value C19 -> Ceramic CAP 0402(1005)
- C20: value C20 -> Ceramic CAP 0402(1005)
- C21: value C21 -> Ceramic CAP 0402(1005)
- C22: value C22 -> Ceramic CAP 0402(1005)
- C23: value C23 -> Ceramic CAP 0402(1005)
- C28: value C28 -> Ceramic CAP 0402(1005)
- C29: value C29 -> Ceramic CAP 0402(1005)
- C30: value C30 -> Ceramic CAP 0402(1005)
- C31: value C31 -> Ceramic CAP 1808(4520)
- C35: value C35 -> Ceramic CAP 0402(1005)
- C36: value C36 -> Ceramic CAP 0402(1005)
- J1: value J1 -> 2.54mm 1x20 Pin Header DIP
- J2: value J2 -> 2.54mm 1x20 Pin Header DIP
- J3: value J3 -> 2.54mm 1x3 Pin Header DIP
- LD2: value LD2 -> LED-0603
- P1: value P1 -> Micro USB B Connector SMD
- P2: value P2 -> J1B1211CCD
- R12: value R12 -> RES-0402
- R15: value R15 -> RES-0402
- R16: value R16 -> RES-0402
- R17: value R17 -> RES-0402
- R18: value R18 -> RES-0402
- R19: value R19 -> RES-0402
- R20: value R20 -> RES-0402
- R21: value R21 -> RES-0402
- R22: value R22 -> RES-0402
- R26: value R26 -> RES-0402
- R27: value R27 -> RES-0402
- R28: value R28 -> RES-0402
- R29: value R29 -> RES-0402
- R3: value R3 -> RES-0402
- R30: value R30 -> RES-0402
- R4: value R4 -> RES-0402
- R5: value R5 -> RES-0402
- moved C12 1252.7 mm to (154.8, 81.9)
- moved C15 1252.7 mm to (131.7, 82.1)
- moved C16 1252.7 mm to (131.7, 81.1)
- moved C17 1252.7 mm to (127.0, 93.6)
- moved C20 1252.7 mm to (127.0, 88.5)
- moved C21 1252.7 mm to (127.0, 91.5)
- moved C28 1252.7 mm to (124.7, 84.5)
- moved C30 1252.7 mm to (124.7, 92.5)
- moved C31 1252.7 mm to (127.2, 82.2)
- moved C35 1252.7 mm to (124.7, 90.5)
- moved C36 1252.7 mm to (124.7, 89.5)
- moved J2 1252.7 mm to (131.5, 97.4)
- moved P1 1252.7 mm to (181.2, 88.5)
- moved P2 1252.7 mm to (104.7, 88.5)
- moved R15 1252.7 mm to (127.0, 86.5)
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Routing:
- net Net1: track 972.8 -> 0.00 mm
- net 3V3: track 187.8 -> 72.4 mm, vias 14 -> 3
- net GND: track 120.6 -> 56.5 mm, vias 79 -> 34
- net GPIO19: track 49.2 -> 12.5 mm, vias 2 -> 0
- net GPIO16: track 42.9 -> 6.72 mm, vias 2 -> 0
- net GPIO17: track 42.3 -> 6.33 mm, vias 2 -> 0
- net GPIO18: track 47.5 -> 12.8 mm, vias 2 -> 0
- net 1V1: track 29.0 -> 0.00 mm, vias 3 -> 0
- net GPIO25: track 25.6 -> 0.00 mm, vias 2 -> 0
- net GPIO20: track 44.8 -> 19.4 mm, vias 3 -> 0
- net GPIO21: track 43.1 -> 18.2 mm, vias 3 -> 1
- net QSPI1_SS_N: track 23.6 -> 0.00 mm, vias 2 -> 0
- net GPIO24: track 22.3 -> 0.00 mm, vias 2 -> 0
- net RUN: track 26.5 -> 5.88 mm, vias 2 -> 0
- net NetR9_2: track 16.8 -> 0.00 mm, vias 2 -> 0
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- removed copper zone on F.Cu, net 3V3
Other:
- net class Default removed
- board text removed: "BOOTSEL"
- board text removed: "C10"
- board text removed: "C14"
- board text removed: "C15"
- board text removed: "C18"
- board text removed: "C2"
- board text removed: "C21"
- board text removed: "C24"
- board text removed: "C26"
- board text removed: "C27"
- board text removed: "C29"
- board text removed: "C32"
- board text removed: "C33"
- board text removed: "C34"
- board text removed: "C37"
- board text removed: "C4"
- board text removed: "C5"
- board text removed: "C6"
- board text removed: "C7"
- board text removed: "C8"
- board text removed: "C9"
- board text removed: "DEBUG"
- board text removed: "J3"
- board text removed: "L1"
- board text removed: "R1"
- board text removed: "R10"
- board text removed: "R13"
- board text removed: "R14"
- board text removed: "R16"
- board text removed: "R17"
- board text removed: "R18"
- board text removed: "R23"
- board text removed: "R24"
- board text removed: "R25"
- board text removed: "R32"
- board text removed: "R33"
- board text removed: "R6"
- board text removed: "R7"
- board text removed: "R8"
- board text removed: "R9"
- board text removed: "SWCLK"
- board text removed: "SWDIO"
- board text removed: "U2"
- board text removed: "U3"
- board text removed: "U4"
- board text removed: "Y2"
