File: hw/pcb_v6/pcb.kicad_pcb (KiCad board)
At the start: 2 copper layers, 100 x 76 mm, 34 parts, among them J1 Barrel_Jack_MountingPin, J3 Conn_01x02, J4 RS232, Q1 DMG2305UX-7, Q2 DMG2305UX-7, SW1 SW_Push, U1 MP1584EN, U2 Raspberry Pi Pico W, U3 MAX3232, U4 W5500-EVB-Pico

Commit message: pcb update
Parts:
- moved SW1 14.7 mm to (23.1, 53.5)
- moved C9 14.6 mm to (23.9, 58.9)
- moved R9 14.6 mm to (23.9, 61.9)
Connections:
- R10 pad 2: Net-(U4-GPIO26_ADC0) -> Net-(U4-GPIO13)
- R7 pad 2: Net-(U4-GPIO28_ADC2) -> Net-(U4-GPIO15)
- R8 pad 2: Net-(U4-GPIO27_ADC1) -> Net-(U4-GPIO14)
- U4 pad 12: unconnected-(U4-GPIO9-Pad12) -> BTN
- U4 pad 17: BTN -> Net-(U4-GPIO13)
- U4 pad 19: unconnected-(U4-GPIO14-Pad19) -> Net-(U4-GPIO14)
- U4 pad 20: unconnected-(U4-GPIO15-Pad20) -> Net-(U4-GPIO15)
- U4 pad 31: Net-(U4-GPIO26_ADC0) -> unconnected-(U4-GPIO26_ADC0-Pad31)
- U4 pad 32: Net-(U4-GPIO27_ADC1) -> unconnected-(U4-GPIO27_ADC1-Pad32)
- U4 pad 34: Net-(U4-GPIO28_ADC2) -> unconnected-(U4-GPIO28_ADC2-Pad34)
Routing:
- net (no net): track 89.3 -> 0.00 mm
- net Net-(D3-A): track 0.00 -> 47.8 mm
- net Net-(D2-A): track 0.00 -> 41.5 mm
- net Net-(U4-GPIO28_ADC2): track 8.33 -> 0.00 mm
- net Net-(U4-GPIO15): track 0.00 -> 8.33 mm
- net Net-(U4-GPIO27_ADC1): track 7.04 -> 0.00 mm
- net Net-(U4-GPIO14): track 0.00 -> 7.04 mm
- net Net-(U4-GPIO13): track 0.00 -> 2.54 mm
- net GND: track 487.8 -> 486.6 mm

Commit message: sch & pcb update
Parts:
- moved R8 50.5 mm to (113.6, 67.1)
- moved R7 50.1 mm to (113.6, 61.1)
- moved D2 12.6 mm to (110.2, 57.7), turned to -90 degrees
- moved D3 12.2 mm to (110.2, 63.7), turned to -90 degrees
- moved D4 11.7 mm to (110.2, 69.7), turned to -90 degrees
- moved R10 6.25 mm to (113.5, 73.0), turned to -90 degrees
- moved J4 0.60 mm to (101.0, 89.5)
Connections:
- D1 pad 2: (no net) -> GND
- R7 pad 2: Net-(U4-GPIO15) -> Net-(U4-GPIO14)
- R8 pad 2: Net-(U4-GPIO14) -> Net-(U4-GPIO15)
Routing:
- net Net-(U4-GPIO14): track 7.04 -> 127.3 mm, vias 0 -> 2
- net Net-(U4-GPIO15): track 8.33 -> 107.0 mm, vias 0 -> 2
- net Net-(U4-GPIO13): track 2.54 -> 99.6 mm, vias 0 -> 2
- net Net-(D3-A): track 47.8 -> 3.35 mm
- net Net-(D2-A): track 41.5 -> 3.35 mm
- net +3.3V: track 135.3 -> 145.5 mm
- net GND: track 486.6 -> 493.8 mm
- net Net-(D4-A): track 0.00 -> 3.30 mm
- net BTN: track 23.9 -> 23.1 mm
- net RS232_TX: track 40.5 -> 39.9 mm
- net RS232_RX: track 43.6 -> 43.0 mm
Other:
- outline, holes or cut-outs redrawn
- board text added: "Robotus v1.0"
