File: hw/pcb_v6/pcb.kicad_sch (KiCad schematic)
At the start: 34 parts, among them J1 Barrel_Jack_MountingPin, J1 RS232, J3 Conn_01x02, Q1 DMG2305UX-7, Q2 DMG2305UX-7, SW1 SW_Push, U1 MP1584EN, U2 Raspberry Pi Pico W, U3 MAX3232, U4 W5500-EVB-Pico

Commit message: sch update
Connections:
- net BTN: now also U4.12 (GPIO9); no longer U4.17 (GPIO13)
- net at R61.2: no longer U4.31 (GPIO26_ADC0)
- net at R61.2: no longer U4.34 (GPIO28_ADC2)
- net at R61.2: no longer U4.32 (GPIO27_ADC1)
- no-connect marks 60 -> 59
Other:
- moved on the sheet: D2, D3, D4, R61

Commit message: pcb update
Connections:
- net at R61.2: now also U4.17 (GPIO13)
- net at R61.2: now also U4.20 (GPIO15)
- net at R61.2: now also U4.19 (GPIO14)
- no-connect marks 59 -> 60
Other:
- moved on the sheet: D2, D3, D4, R61

Commit message: sch & pcb update
Connections:
- net at R61.2: now also U4.19 (GPIO14); no longer U4.20 (GPIO15)
- net at R61.2: now also U4.20 (GPIO15); no longer U4.19 (GPIO14)
Other:
- moved on the sheet: D2, D3, R61

Commit message: pcb v6.2 submitted to jlcpcb
Parts:
- J1: LCSC C141880 -> (none)
- R1: LCSC C25271 -> C149504
- R61: LCSC C4190 -> C22787
Changed lines of the file:
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@@
       (effects (font (size 1.27 1.27)) hide)
     )
-    (property "LCSC" "C4190" (at 109.22 186.69 0)
+    (property "LCSC" "C22787" (at 109.22 186.69 0)
       (effects (font (size 1.27 1.27)) hide)
     )
@@
       (effects (font (size 1.27 1.27)) hide)
     )
-    (property "LCSC" "C141880" (at 257.81 46.99 0)
+    (property "LCSC" "" (at 257.81 46.99 0)
       (effects (font (size 1.27 1.27)) hide)
     )
@@
       (effects (font (size 1.27 1.27)) hide)
     )
-    (property "LCSC" "C4190" (at 109.22 177.8 0)
+    (property "LCSC" "C22787" (at 109.22 177.8 0)
       (effects (font (size 1.27 1.27)) hide)
     )
@@
       (effects (font (size 1.27 1.27)) hide)
     )
-    (property "LCSC" "C4190" (at 109.22 168.91 0)
+    (property "LCSC" "C22787" (at 109.22 168.91 0)
       (effects (font (size 1.27 1.27)) hide)
     )
@@
       (effects (font (size 1.27 1.27)) hide)
     )
-    (property "LCSC" "C25271" (at 80.01 40.64 0)
-      (effects (font (size 1.27 1.27)) hide)
-    )
+    (property "LCSC" "C149504" (at 80.01 40.64 0)
+      (effects (font (size 1.27 1.27)) hide)
+    )
